File: PCB/BatPad.kicad_pcb (KiCad board)
At the start: 2 copper layers, 95 x 60 mm, 10 parts, among them SW1 SW_Push, SW2 SW_Push, SW3 SW_Push, SW4 SW_Push, SW5 RotaryEncoder, SW6 RotaryEncoder, U1 XIAO-RP2040-DIP

Commit message: fixed schematic (gnd anf 5v)
Connections:
- U1 pad 13: unconnected-(U1-GND-Pad13) -> GND
- U1 pad 14: unconnected-(U1-VBUS-Pad14) -> +5V
Routing:
- net +5V: track 64.2 -> 119.2 mm
- net Net-(U1-GPIO28/ADC2/A2): track 107.1 -> 70.8 mm
- net GND: track 218.9 -> 254.4 mm
Changed lines of the file:
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@@
 	(net 9 "Net-(U1-GPIO1{slash}RX)")
 	(net 10 "unconnected-(U1-GPIO0{slash}TX-Pad7)")
-	(net 11 "unconnected-(U1-VBUS-Pad14)")
-	(net 12 "unconnected-(U1-3V3-Pad12)")
-	(net 13 "unconnected-(U1-GND-Pad13)")
-	(net 14 "unconnected-(U1-GPIO26{slash}ADC0{slash}A0-Pad1)")
-	(net 15 "Net-(U1-GPIO28{slash}ADC2{slash}A2)")
-	(net 16 "Net-(U1-GPIO7{slash}SCL)")
-	(net 17 "Net-(U1-GPIO29{slash}ADC3{slash}A3)")
-	(net 18 "Net-(U1-GPIO27{slash}ADC1{slash}A1)")
+	(net 11 "unconnected-(U1-3V3-Pad12)")
+	(net 12 "unconnected-(U1-GPIO26{slash}ADC0{slash}A0-Pad1)")
+	(net 13 "Net-(U1-GPIO28{slash}ADC2{slash}A2)")
+	(net 14 "Net-(U1-GPIO7{slash}SCL)")
+	(net 15 "Net-(U1-GPIO29{slash}ADC3{slash}A3)")
+	(net 16 "Net-(U1-GPIO27{slash}ADC1{slash}A1)")
 	(footprint "LED_SMD:LED_SK6812MINI_PLCC4_3.5x3.5mm_P1.75mm"
 		(layer "F.Cu")
@@
 			(layers "*.Cu" "*.Mask")
 			(remove_unused_layers no)
-			(net 15 "Net-(U1-GPIO28{slash}ADC2{slash}A2)")
+			(net 13 "Net-(U1-GPIO28{slash}ADC2{slash}A2)")
 			(pinfunction "A")
 			(pintype "passive")
@@
 			(layers "*.Cu" "*.Mask")
 			(remove_unused_layers no)
-			(net 18 "Net-(U1-GPIO27{slash}ADC1{slash}A1)")
+			(net 16 "Net-(U1-GPIO27{slash}ADC1{slash}A1)")
 			(pinfunction "B")
 			(pintype "passive")
@@
 			(layers "*.Cu" "*.Mask")
 			(remove_unused_layers no)
-			(net 16 "Net-(U1-GPIO7{slash}SCL)")
+			(net 14 "Net-(U1-GPIO7{slash}SCL)")
 			(pinfunction "A")
 			(pintype "passive")
@@
 			(layers "*.Cu" "*.Mask")
 			(remove_unused_layers no)
-			(net 17 "Net-(U1-GPIO29{slash}ADC3{slash}A3)")
+			(net 15 "Net-(U1-GPIO29{slash}ADC3{slash}A3)")
 			(pinfunction "B")
 			(pintype "passive")
@@
 			(layers "F.Cu" "F.Mask")
 			(roundrect_rratio 0.1)
-			(net 14 "unconnected-(U1-GPIO26{slash}ADC0{slash}A0-Pad1)")
+			(net 12 "unconnected-(U1-GPIO26{slash}ADC0{slash}A0-Pad1)")
 			(pinfunction "GPIO26/ADC0/A0")
 			(pintype "passive")
@@
 			(layers "*.Cu" "*.Mask")
 			(remove_unused_layers no)
-			(net 14 "unconnected-(U1-GPIO26{slash}ADC0{slash}A0-Pad1)")
+			(net 12 "unconnected-(U1-GPIO26{slash}ADC0{slash}A0-Pad1)")
 			(pinfunction "GPIO26/ADC0/A0")
 			(pintype "passive")
@@
 			(layers "F.Cu" "F.Mask")
 			(roundrect_rratio 0.1)
-			(net 18 "Net-(U1-GPIO27{slash}ADC1{slash}A1)")
+			(net 16 "Net-(U1-GPIO27{slash}ADC1{slash}A1)")
 			(pinfunction "GPIO27/ADC1/A1")
 			(pintype "passive")
@@
 			(layers "*.Cu" "*.Mask")
 			(remove_unused_layers no)
-			(net 18 "Net-(U1-GPIO27{slash}ADC1{slash}A1)")
+			(net 16 "Net-(U1-GPIO27{slash}ADC1{slash}A1)")
 			(pinfunction "GPIO27/ADC1/A1")
 			(pintype "passive")
@@
 			(layers "F.Cu" "F.Mask")
 			(roundrect_rratio 0.1)
-			(net 15 "Net-(U1-GPIO28{slash}ADC2{slash}A2)")
+			(net 13 "Net-(U1-GPIO28{slash}ADC2{slash}A2)")
 			(pinfunction "GPIO28/ADC2/A2")
 			(pintype "passive")
@@
 			(layers "*.Cu" "*.Mask")
 			(remove_unused_layers no)
-			(net 15 "Net-(U1-GPIO28{slash}ADC2{slash}A2)")
+			(net 13 "Net-(U1-GPIO28{slash}ADC2{slash}A2)")
 			(pinfunction "GPIO28/ADC2/A2")
 			(pintype "passive")
@@
 			(layers "F.Cu" "F.Mask")
 			(roundrect_rratio 0.1)
-			(net 17 "Net-(U1-GPIO29{slash}ADC3{slash}A3)")
+			(net 15 "Net-(U1-GPIO29{slash}ADC3{slash}A3)")
 			(pinfunction "GPIO29/ADC3/A3")
 			(pintype "passive")
@@
 			(layers "*.Cu" "*.Mask")
 			(remove_unused_layers no)
-			(net 17 "Net-(U1-GPIO29{slash}ADC3{slash}A3)")
+			(net 15 "Net-(U1-GPIO29{slash}ADC3{slash}A3)")
 			(pinfunction "GPIO29/ADC3/A3")
 			(pintype "passive")
@@
 			(layers "F.Cu" "F.Mask")
 			(roundrect_rratio 0.1)
-			(net 16 "Net-(U1-GPIO7{slash}SCL)")
+			(net 14 "Net-(U1-GPIO7{slash}SCL)")
 			(pinfunction "GPIO7/SCL")
 			(pintype "passive")
@@
 			(layers "*.Cu" "*.Mask")
 			(remove_unused_layers no)
-			(net 16 "Net-(U1-GPIO7{slash}SCL)")
+			(net 14 "Net-(U1-GPIO7{slash}SCL)")
 			(pinfunction "GPIO7/SCL")
 			(pintype "passive")
@@
 			(layers "*.Cu" "*.Mask")
 			(remove_unused_layers no)
-			(net 12 "unconnected-(U1-3V3-Pad12)")
+			(net 11 "unconnected-(U1-3V3-Pad12)")
 			(pinfunction "3V3")
 			(pintype "passive")
@@
 			(layers "F.Cu" "F.Mask")
 			(roundrect_rratio 0.1)
-			(net 12 "unconnected-(U1-3V3-Pad12)")
+			(net 11 "unconnected-(U1-3V3-Pad12)")
 			(pinfunction "3V3")
 			(pintype "passive")
@@
 			(layers "*.Cu" "*.Mask")
 			(remove_unused_layers no)
-			(net 13 "unconnected-(U1-GND-Pad13)")
+			(net 1 "GND")
 			(pinfunction "GND")
 			(pintype "passive")
@@
 			(layers "F.Cu" "F.Mask")
 			(roundrect_rratio 0.1)
-			(net 13 "unconnected-(U1-GND-Pad13)")
+			(net 1 "GND")
 			(pinfunction "GND")
 			(pintype "passive")
@@
 			(layers "*.Cu" "*.Mask")
 			(remove_unused_layers no)
-			(net 11 "unconnected-(U1-VBUS-Pad14)")
+			(net 2 "+5V")
 			(pinfunction "VBUS")
 			(pintype "passive")
@@
 			(layers "F.Cu" "F.Mask")
 			(roundrect_rratio 0.1)
-			(net 11 "unconnected-(U1-VBUS-Pad14)")
+			(net 2 "+5V")
 			(pinfunction "VBUS")
 			(pintype "passive")
@@
 	)
 	(segment
+		(start 40.262756 54.320625)
+		(end 41.325756 53.257625)
+		(width 0.2)
+		(layer "B.Cu")
+		(net 1)
+	)
+	(segment
 		(start 64.817934 27.861)
 		(end 68.758934 23.92)
@@
 	)
 	(segment
+		(start 40.703066 47.763625)
+		(end 39.822446 47.763625)
+		(width 0.2)
+		(layer "B.Cu")
+		(net 1)
+	)
+	(segment
 		(start 61.79275 14.61525)
 		(end 61.79275 27.040314)
@@
 	)
 	(segment
+		(start 41.325756 48.386315)
+		(end 40.703066 47.763625)
+		(width 0.2)
+		(layer "B.Cu")
+		(net 1)
+	)
+	(segment
 		(start 58.04165 8.12925)
 		(end 50.46 15.7109)
@@
 	)
 	(segment
+		(start 31.41375 39.354929)
+		(end 31.41375 23.92)
+		(width 0.2)
+		(layer "B.Cu")
+		(net 1)
+	)
+	(segment
+		(start 41.325756 53.257625)
+		(end 41.325756 48.386315)
+		(width 0.2)
+		(layer "B.Cu")
+		(net 1)
+	)
+	(segment
 		(start 50.46 15.7109)
 		(end 50.46 23.92)
@@
 	)
 	(segment
+		(start 39.822446 47.763625)
+		(end 31.41375 39.354929)
+		(width 0.2)
+		(layer "B.Cu")
+		(net 1)
+	)
+	(segment
+		(start 41.325756 57.923625)
+		(end 63.4261 57.923625)
+		(width 0.2)
+		(layer "F.Cu")
+		(net 2)
+	)
+	(segment
+		(start 82.20285 35.646875)
+		(end 81.55875 35.646875)
+		(width 0.2)
+		(layer "F.Cu")
+		(net 2)
+	)
+	(segment
+		(start 83.06075 36.504775)
+		(end 82.20285 35.646875)
+		(width 0.2)
+		(layer "F.Cu")
+		(net 2)
+	)
+	(segment
 		(start 17.95875 35.596875)
 		(end 18.63475 34.920875)
@@
 	)
 	(segment
+		(start 83.06075 38.288975)
+		(end 83.06075 36.504775)
+		(width 0.2)
+		(layer "F.Cu")
+		(net 2)
+	)
+	(segment
+		(start 40.262756 56.860625)
+		(end 41.325756 57.923625)
+		(width 0.2)
+		(layer "F.Cu")
+		(net 2)
+	)
+	(segment
+		(start 63.4261 57.923625)
+		(end 83.06075 38.288975)
+		(width 0.2)
+		(layer "F.Cu")
+		(net 2)
+	)
+	(segment
 		(start 18.63475 34.920875)
 		(end 80.83275 34.920875)
@@
 	)
 	(segment
-		(start 56.28875 51.780625)
-		(end 69.5691 51.780625)
+		(start 22.59275 15.877767)
+		(end 23.23475 15.235767)
 		(width 0.2)
-		(layer "F.Cu")
-		(net 15)
+		(layer "B.Cu")
+		(net 13)
 	)
 	(segment
-		(start 34.071125 19.23225)
-		(end 24.53575 9.696875)
+		(start 22.59275 38.153929)
+		(end 22.59275 15.877767)
 		(width 0.2)
-		(layer "F.Cu")
-		(net 15)
+		(layer "B.Cu")
+		(net 13)
 	)
 	(segment
-		(start 83.06075 35.321875)
-		(end 66.971125 19.23225)
+		(start 23.23475 15.235767)
+		(end 23.23475 10.997875)
 		(width 0.2)
-		(layer "F.Cu")
-		(net 15)
+		(layer "B.Cu")
+		(net 13)
 	)
 	(segment
-		(start 69.5691 51.780625)
-		(end 83.06075 38.288975)
+		(start 23.23475 10.997875)
+		(end 21.93375 9.696875)
 		(width 0.2)
-		(layer "F.Cu")
-		(net 15)
+		(layer "B.Cu")
+		(net 13)
 	)
 	(segment
-		(start 24.53575 9.696875)
-		(end 21.93375 9.696875)
+		(start 55.502756 51.780625)
+		(end 51.899756 55.383625)
 		(width 0.2)
-		(layer "F.Cu")
-		(net 15)
+		(layer "B.Cu")
+		(net 13)
 	)
 	(segment
-		(start 83.06075 38.288975)
-		(end 83.06075 35.321875)
+		(start 51.899756 55.383625)
+		(end 39.822446 55.383625)
 		(width 0.2)
-		(layer "F.Cu")
-		(net 15)
+		(layer "B.Cu")
+		(net 13)
 	)
 	(segment
-		(start 66.971125 19.23225)
-		(end 34.071125 19.23225)
+		(start 39.822446 55.383625)
+		(end 22.59275 38.153929)
 		(width 0.2)
-		(layer "F.Cu")
-		(net 15)
+		(layer "B.Cu")
+		(net 13)
 	)
 	(segment
@@
 		(width 0.2)
 		(layer "B.Cu")
-		(net 16)
+		(net 14)
 	)
 	(segment
@@
 		(width 0.2)
 		(layer "B.Cu")
-		(net 16)
+		(net 14)
 	)
 	(segment
@@
 		(width 0.2)
 		(layer "B.Cu")
-		(net 16)
+		(net 14)
 	)
 	(segment
@@
 		(width 0.2)
 		(layer "B.Cu")
-		(net 17)
+		(net 15)
 	)
 	(segment
@@
 		(width 0.2)
 		(layer "B.Cu")
-		(net 17)
+		(net 15)
 	)
 	(segment
@@
 		(width 0.2)
 		(layer "B.Cu")
-		(net 17)
+		(net 15)
 	)
 	(segment
@@
 		(width 0.2)
 		(layer "F.Cu")
-		(net 18)
+		(net 16)
 	)
 	(segment
@@
 		(width 0.2)
 		(layer "F.Cu")
-		(net 18)
+		(net 16)
 	)
 	(segment
@@
 		(width 0.2)
 		(layer "F.Cu")
-		(net 18)
+		(net 16)
 	)
 	(segment
@@
 		(width 0.2)
 		(layer "F.Cu")
-		(net 18)
+		(net 16)
 	)
 	(segment
@@
 		(width 0.2)
 		(layer "F.Cu")
-		(net 18)
+		(net 16)
 	)
 	(embedded_fonts no)
